File: ConPower.kicad_sch (KiCad schematic)
At the start: 81 parts, among them J4 Conn_02x06_Odd_Even, J8 Conn_01x04_Male, U4 4040, U5 4040, U6 TPS65130RGE

Commit message: add counter reset button + cleanup
Parts:
- added R58: 1k, Resistor_SMD:R_0402_1005Metric, symbol Device:R
- added SW1: SW_Push_Dual, Button_Switch_SMD:SW_DIP_SPSTx01_Slide_6.7x4.1mm_W8.61mm_P2.54mm_LowProfile, symbol Switch:SW_Push
Connections:
- net +3.3V: now also SW1.1
- net GND: now also R58.1; no longer U4.11 (Reset), U5.11 (Reset)
- new net: R58.2, SW1.2, U4.11 (Reset), U5.11 (Reset)
Changed lines of the file:
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@@
   (junction (at 244.475 86.995) (diameter 0) (color 0 0 0 0)
   )
+  (junction (at 52.07 125.095) (diameter 0) (color 0 0 0 0)
+  )
   (junction (at 228.6 67.945) (diameter 0) (color 0 0 0 0)
   )
@@
   (junction (at 155.575 85.725) (diameter 0) (color 0 0 0 0)
   )
+  (junction (at 48.26 125.095) (diameter 0) (color 0 0 0 0)
+  )
   (junction (at 208.915 76.2) (diameter 0) (color 0 0 0 0)
   )
@@
   (junction (at 132.08 108.585) (diameter 0) (color 0 0 0 0)
   )
+  (wire (pts (xy 48.26 125.095) (xy 52.07 125.095))
+    (stroke (width 0) (type default) (color 0 0 0 0))
+  )
   (wire (pts (xy 199.39 76.2) (xy 199.39 74.93))
     (stroke (width 0) (type default) (color 0 0 0 0))
@@
     (stroke (width 0) (type default) (color 0 0 0 0))
   )
-  (wire (pts (xy 55.245 127.635) (xy 55.245 125.095))
+  (wire (pts (xy 52.07 98.425) (xy 109.22 98.425))
     (stroke (width 0) (type default) (color 0 0 0 0))
   )
@@
     (stroke (width 0) (type default) (color 0 0 0 0))
   )
+  (wire (pts (xy 48.26 132.715) (xy 48.26 134.62))
+    (stroke (width 0) (type default) (color 0 0 0 0))
+  )
   (wire (pts (xy 217.17 103.505) (xy 227.965 103.505))
     (stroke (width 0) (type default) (color 0 0 0 0))
@@
     (stroke (width 0) (type default) (color 0 0 0 0))
   )
+  (wire (pts (xy 109.22 127) (xy 119.38 127))
+    (stroke (width 0) (type default) (color 0 0 0 0))
+  )
   (wire (pts (xy 68.58 153.035) (xy 68.58 154.94))
     (stroke (width 0) (type default) (color 0 0 0 0))
@@
     (stroke (width 0) (type default) (color 0 0 0 0))
   )
-  (wire (pts (xy 55.245 125.095) (xy 55.88 125.095))
+  (wire (pts (xy 43.18 125.095) (xy 48.26 125.095))
     (stroke (width 0) (type default) (color 0 0 0 0))
   )
@@
     (stroke (width 0) (type default) (color 0 0 0 0))
   )
+  (wire (pts (xy 109.22 98.425) (xy 109.22 127))
+    (stroke (width 0) (type default) (color 0 0 0 0))
+  )
   (wire (pts (xy 240.665 83.82) (xy 240.665 88.265))
     (stroke (width 0) (type default) (color 0 0 0 0))
@@
     (stroke (width 0) (type default) (color 0 0 0 0))
   )
+  (wire (pts (xy 29.21 125.095) (xy 33.02 125.095))
+    (stroke (width 0) (type default) (color 0 0 0 0))
+  )
   (wire (pts (xy 175.26 67.945) (xy 176.53 67.945))
     (stroke (width 0) (type default) (color 0 0 0 0))
@@
     (stroke (width 0) (type default) (color 0 0 0 0))
   )
+  (wire (pts (xy 52.07 125.095) (xy 52.07 98.425))
+    (stroke (width 0) (type default) (color 0 0 0 0))
+  )
   (wire (pts (xy 93.98 75.565) (xy 81.28 75.565))
     (stroke (width 0) (type default) (color 0 0 0 0))
@@
     (stroke (width 0) (type default) (color 0 0 0 0))
   )
-  (wire (pts (xy 118.745 127) (xy 119.38 127))
-    (stroke (width 0) (type default) (color 0 0 0 0))
-  )
   (wire (pts (xy 208.915 62.865) (xy 212.09 62.865))
     (stroke (width 0) (type default) (color 0 0 0 0))
@@
     (stroke (width 0) (type default) (color 0 0 0 0))
   )
+  (wire (pts (xy 29.21 122.555) (xy 29.21 125.095))
+    (stroke (width 0) (type default) (color 0 0 0 0))
+  )
   (wire (pts (xy 176.53 88.265) (xy 176.53 90.805))
     (stroke (width 0) (type default) (color 0 0 0 0))
@@
     (stroke (width 0) (type default) (color 0 0 0 0))
   )
-  (wire (pts (xy 118.745 129.54) (xy 118.745 127))
+  (wire (pts (xy 52.07 125.095) (xy 55.88 125.095))
     (stroke (width 0) (type default) (color 0 0 0 0))
   )
@@
     )
     (pin "1")
+  )
+  (symbol (lib_id "Switch:SW_Push") (at 38.1 125.095 0) (unit 1)
+    (in_bom yes) (on_board yes) (fields_autoplaced)
+    (property "Reference" "SW1" (id 0) (at 38.1 118.4742 0))
+    (property "Value" "SW_Push_Dual" (id 1) (at 38.1 121.0111 0))
+    (property "Footprint" "Button_Switch_SMD:SW_DIP_SPSTx01_Slide_6.7x4.1mm_W8.61mm_P2.54mm_LowProfile" (id 2) (at 38.1 120.015 0)
+      (effects (font (size 1.27 1.27)) hide)
+    )
+    (property "Datasheet" "~" (id 3) (at 38.1 120.015 0)
+      (effects (font (size 1.27 1.27)) hide)
+    )
+    (pin "1")
+    (pin "2")
   )
   (symbol (lib_id "power:GND") (at 186.69 107.315 0) (unit 1)
@@
     (pin "2")
   )
-  (symbol (lib_id "power:GND") (at 55.245 127.635 0) (unit 1)
-    (in_bom yes) (on_board yes) (fields_autoplaced)
-    (property "Reference" "#PWR0149" (id 0) (at 55.245 133.985 0)
-      (effects (font (size 1.27 1.27)) hide)
-    )
-    (property "Value" "GND" (id 1) (at 55.245 132.0784 0))
-    (property "Footprint" "" (id 2) (at 55.245 127.635 0)
-      (effects (font (size 1.27 1.27)) hide)
-    )
-    (property "Datasheet" "" (id 3) (at 55.245 127.635 0)
+  (symbol (lib_id "power:GND") (at 48.26 134.62 0) (unit 1)
+    (in_bom yes) (on_board yes) (fields_autoplaced)
+    (property "Reference" "#PWR0149" (id 0) (at 48.26 140.97 0)
+      (effects (font (size 1.27 1.27)) hide)
+    )
+    (property "Value" "GND" (id 1) (at 48.26 139.0634 0))
+    (property "Footprint" "" (id 2) (at 48.26 134.62 0)
+      (effects (font (size 1.27 1.27)) hide)
+    )
+    (property "Datasheet" "" (id 3) (at 48.26 134.62 0)
       (effects (font (size 1.27 1.27)) hide)
     )
@@
     (pin "2")
   )
+  (symbol (lib_id "power:+3.3V") (at 29.21 122.555 0) (unit 1)
+    (in_bom yes) (on_board yes) (fields_autoplaced)
+    (property "Reference" "#PWR0146" (id 0) (at 29.21 126.365 0)
+      (effects (font (size 1.27 1.27)) hide)
+    )
+    (property "Value" "+3.3V" (id 1) (at 29.21 118.9792 0))
+    (property "Footprint" "" (id 2) (at 29.21 122.555 0)
+      (effects (font (size 1.27 1.27)) hide)
+    )
+    (property "Datasheet" "" (id 3) (at 29.21 122.555 0)
+      (effects (font (size 1.27 1.27)) hide)
+    )
+    (pin "1")
+  )
   (symbol (lib_id "Device:R") (at 148.59 144.78 90) (unit 1)
     (in_bom yes) (on_board yes) (fields_autoplaced)
@@
     (pin "1")
   )
+  (symbol (lib_id "Device:R") (at 48.26 128.905 180) (unit 1)
+    (in_bom yes) (on_board yes) (fields_autoplaced)
+    (property "Reference" "R58" (id 0) (at 50.038 128.0703 0)
+      (effects (font (size 1.27 1.27)) (justify right))
+    )
+    (property "Value" "1k" (id 1) (at 50.038 130.6072 0)
+      (effects (font (size 1.27 1.27)) (justify right))
+    )
+    (property "Footprint" "Resistor_SMD:R_0402_1005Metric" (id 2) (at 50.038 128.905 90)
+      (effects (font (size 1.27 1.27)) hide)
+    )
+    (property "Datasheet" "~" (id 3) (at 48.26 128.905 0)
+      (effects (font (size 1.27 1.27)) hide)
+    )
+    (pin "1")
+    (pin "2")
+  )
   (symbol (lib_id "power:GND") (at 160.02 151.13 0) (unit 1)
     (in_bom yes) (on_board yes) (fields_autoplaced)
@@
     (pin "2")
   )
-  (symbol (lib_id "power:GND") (at 118.745 129.54 0) (unit 1)
-    (in_bom yes) (on_board yes) (fields_autoplaced)
-    (property "Reference" "#PWR0146" (id 0) (at 118.745 135.89 0)
-      (effects (font (size 1.27 1.27)) hide)
-    )
-    (property "Value" "GND" (id 1) (at 118.745 133.9834 0))
-    (property "Footprint" "" (id 2) (at 118.745 129.54 0)
-      (effects (font (size 1.27 1.27)) hide)
-    )
-    (property "Datasheet" "" (id 3) (at 118.745 129.54 0)
-      (effects (font (size 1.27 1.27)) hide)
-    )
-    (pin "1")
-  )
   (symbol (lib_id "power:+3.3V") (at 155.575 67.31 0) (unit 1)
